Commit message: First launchable version

File: src/jackal_custom/urdf/jackal.urdf (robot description, URDF)
Before this commit: robot jackal, 19 links, 18 joints
Links:
- link base_link: geometry collision box size=0.42 0.31 0.184; visual mesh filename=file:///workspaces/2022-TUB-MARS-autopilot/src/jackal_custo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
- link front_fender_link: geometry collision mesh filename=file:///workspaces/2022-TUB-MARS-autopilot/src/jackal_custo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; visual mesh filename=file:///workspaces/2022-TUB-MARS-autopilot/src/jackal_custo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
- link front_left_wheel_link: geometry collision cylinder length=0.04 radius=0.098; visual mesh filename=file:///workspaces/2022-TUB-MARS-autopilot/src/jackal_custo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
- link front_right_wheel_link: geometry collision cylinder length=0.04 radius=0.098; visual mesh filename=file:///workspaces/2022-TUB-MARS-autopilot/src/jackal_custo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
- link imu_link: mass 0.001 -> 0.010
- link laser_link: geometry collision box size=0.105 0.1 0.1; visual mesh filename=file:///workspaces/2022-TUB-MARS-autopilot/src/jackal_custo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
- link laser_mount: geometry visual mesh filename=file:///workspaces/2022-TUB-MARS-autopilot/src/jackal_custo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
- link rear_fender_link: geometry collision mesh filename=file:///workspaces/2022-TUB-MARS-autopilot/src/jackal_custo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; visual mesh filename=file:///workspaces/2022-TUB-MARS-autopilot/src/jackal_custo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
- link rear_left_wheel_link: geometry collision cylinder length=0.04 radius=0.098; visual mesh filename=file:///workspaces/2022-TUB-MARS-autopilot/src/jackal_custo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
- link rear_right_wheel_link: geometry collision cylinder length=0.04 radius=0.098; visual mesh filename=file:///workspaces/2022-TUB-MARS-autopilot/src/jackal_custo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
