Commit message: latest version robot description

File: src/mars_robot/urdf/mars_robot.urdf (robot description, URDF)
Before this commit: robot mars_robot, 9 links, 8 joints
Links:
- link camera_link: geometry visual box size=0.03 0.11 0.035
- link front_left_wheel_link: geometry collision cylinder length=0.068 radius=0.0615; visual cylinder length=0.068 radius=0.0615
- link front_right_wheel_link: geometry collision cylinder length=0.068 radius=0.0615; visual cylinder length=0.068 radius=0.0615
- link rear_left_wheel_link: geometry collision cylinder length=0.068 radius=0.0615; visual cylinder length=0.068 radius=0.0615
- link rear_right_wheel_link: geometry collision cylinder length=0.068 radius=0.0615; visual cylinder length=0.068 radius=0.0615
- link robot_base_link: geometry collision box size=0.326 0.2142 0.300; visual box size=0.326 0.2142 0.175
Joints:
- joint base_joint: origin xyz=0 0 0 rpy=0 0 0 -> xyz=0.0 0 0.0615 rpy=0 0 0
- joint camera_joint: origin xyz=0.0 0 0.2045 rpy=0 0 0 -> xyz=0.1335 0 0.2045 rpy=0 0 0
- joint front_left_wheel_joint: origin xyz=0.13675 0.141 0 rpy=0 0 0 -> xyz=0.0955 0.141 0 rpy=1.5708 0 0
- joint front_right_wheel_joint: origin xyz=0.13675 -0.141 0 rpy=0 0 0 -> xyz=0.0955 -0.141 0 rpy=1.5708 0 0
- joint rear_left_wheel_joint: origin xyz=-0.05425 0.141 0 rpy=0 0 0 -> xyz=-0.0955 0.141 0 rpy=1.5708 0 0
- joint rear_right_wheel_joint: origin xyz=-0.05425 -0.141 0 rpy=0 0 0 -> xyz=-0.0955 -0.141 0 rpy=1.5708 0 0

File: src/mars_robot/urdf/mars_robot.urdf.xacro (robot description, xacro)
@@ -6,9 +6,9 @@
 <link name="robot_base_link">
         <visual>
-                <origin xyz="0 0 0" rpy="0.0 0.0 0.0"/>
+                <origin xyz="0 0 0.1115" rpy="0.0 0.0 0.0"/>
                 <geometry>
                         <!-- <mesh filename="file:///workspaces/2022-TUB-MARS-autopilot/src/mars_robot/meshes/Robot_base.stl"
                         scale="0.001 0.001 0.001"/>            -->
-                        <box size="0.1 0.1 0.1"/>
+                        <box size="0.326 0.2142 0.175"/>
                 </geometry>
                 <material name="red">
@@ -25,7 +25,7 @@
         </inertial>
         <collision>
-                <origin xyz="0.0 0.0 0.0" rpy="0.0 0.0 0.0"/>
-                <geometry>
-                        <box size="0.330 0.355 0.300"/>
+                <origin xyz="0 0 0.1115" rpy="0 0 0"/>
+                <geometry>
+                        <box size="0.326 0.2142 0.300"/>
                 </geometry>
         </collision>
@@ -34,5 +34,5 @@
 <joint name="base_joint" type="fixed">
         <preserveFixedJoint>true</preserveFixedJoint>
-        <origin xyz="0 0 0" rpy="0 0 0"/>
+        <origin xyz="0.0 0 0.0615" rpy="0 0 0"/>
         <parent link="mars_robot_footprint"/>
         <child link="robot_base_link"/>
@@ -44,14 +44,14 @@
                         <!-- <mesh filename="file:///workspaces/2022-TUB-MARS-autopilot/src/mars_robot/meshes/Wheel_one.stl"
                         scale="0.001 0.001 0.001"/> -->
-                        <box size="0.128 0.084 0.061" />
-                </geometry>
-                <material name="color_wheel">
-                <color rgba="0.0 0.0 0.0 1.0"/>
-                </material>
-        </visual>
-        <collision>
-                <origin rpy="0 0 0" xyz="0 0 0" />
-                <geometry>
-                        <cylinder length="0.07" radius="0.125" />
+                        <cylinder length="0.068" radius="0.0615" />
+                </geometry>
+                <material name="color_wheel">
+                <color rgba="0.0 0.0 0.0 1.0"/>
+                </material>
+        </visual>
+        <collision>
+                <origin rpy="0 0 0" xyz="0 0 0" />
+                <geometry>
+                        <cylinder length="0.068" radius="0.0615" />
                 </geometry>
         </collision>
@@ -67,5 +67,5 @@
         <parent link="robot_base_link"/>
         <child link="front_left_wheel_link"/>
-        <origin rpy="0 0 0" xyz="0.13675 0.141 0"/>
+        <origin rpy="1.5708 0 0" xyz="0.0955 0.141 0"/>
         <implicitSpringDamper>1</implicitSpringDamper>
 </joint>
@@ -76,14 +76,14 @@
                         <!-- <mesh filename="file:///workspaces/2022-TUB-MARS-autopilot/src/mars_robot/meshes/Wheel_two.stl"
                         scale="0.001 0.001 0.001"/> -->
-                        <box size="0.128 0.084 0.061" />
-                </geometry>
-                <material name="color_wheel">
-                <color rgba="0.0 0.0 0.0 1.0"/>
-                </material>
-        </visual>
-        <collision>
-                <origin rpy="0 0 0" xyz="0 0 0" />
-                <geometry>
-                        <cylinder length="0.07" radius="0.125" />
+                        <cylinder length="0.068" radius="0.0615" />
+                </geometry>
+                <material name="color_wheel">
+                <color rgba="0.0 0.0 0.0 1.0"/>
+                </material>
+        </visual>
+        <collision>
+                <origin rpy="0 0 0" xyz="0 0 0" />
+                <geometry>
+                        <cylinder length="0.068" radius="0.0615" />
                 </geometry>
         </collision>
@@ -99,5 +99,5 @@
         <parent link="robot_base_link"/>
         <child link="front_right_wheel_link"/>
-        <origin rpy="0 0 0" xyz="0.13675 -0.141 0"/>
+        <origin rpy="1.5708 0 0" xyz="0.0955 -0.141 0"/>
         <implicitSpringDamper>1</implicitSpringDamper>
 </joint>
@@ -108,5 +108,5 @@
                         <!-- <mesh filename="file:///workspaces/2022-TUB-MARS-autopilot/src/mars_robot/meshes/Wheel_three.stl"
                         scale="0.001 0.001 0.001"/> -->
-                        <box size="0.128 0.084 0.061" />
+                        <cylinder length="0.068" radius="0.0615" />
                 </geometry>
                 <material name="color_wheel">
@@ -117,5 +117,5 @@
                 <origin rpy="0 0 0" xyz="0 0 0" />
                         <geometry>
-                        <cylinder length="0.07" radius="0.125" />
+                        <cylinder length="0.068" radius="0.0615" />
                 </geometry>
         </collision>
@@ -131,5 +131,5 @@
         <parent link="robot_base_link"/>
         <child link="rear_left_wheel_link"/>
-        <origin rpy="0 0 0" xyz="-0.05425 0.141 0"/>
+        <origin rpy="1.5708 0 0" xyz="-0.0955 0.141 0"/>
         <implicitSpringDamper>1</implicitSpringDamper>
 </joint>
@@ -140,14 +140,14 @@
                         <!-- <mesh filename="file:///workspaces/2022-TUB-MARS-autopilot/src/mars_robot/meshes/Wheel_four.stl"
                         scale="0.001 0.001 0.001"/> -->
-                        <box size="0.128 0.084 0.061" />
-                </geometry>
-                <material name="color_wheel">
-                <color rgba="0.0 0.0 0.0 1.0"/>
-                </material>
-        </visual>
-        <collision>
-                <origin rpy="0 0 0" xyz="0 0 0" />
-                <geometry>
-                        <cylinder length="0.07" radius="0.125" />
+                        <cylinder length="0.068" radius="0.0615" />
+                </geometry>
+                <material name="color_wheel">
+                <color rgba="0.0 0.0 0.0 1.0"/>
+                </material>
+        </visual>
+        <collision>
+                <origin rpy="0 0 0" xyz="0 0 0" />
+                <geometry>
+                        <cylinder length="0.068" radius="0.0615" />
                 </geometry>
         </collision>
@@ -163,5 +163,5 @@
         <parent link="robot_base_link"/>
         <child link="rear_right_wheel_link"/>
-        <origin rpy="0 0 0" xyz="-0.05425 -0.141 0"/>
+        <origin rpy="1.5708 0 0" xyz="-0.0955 -0.141 0"/>
         <implicitSpringDamper>1</implicitSpringDamper>
 </joint>
@@ -184,8 +184,8 @@
         <visual>
                 <geometry>
-                        <box size="0.128 0.084 0.061" />
+                        <box size="0.03 0.11 0.035"/>
                 </geometry>
                 <material name="color_cam">
-                <color rgba="0.0 0.0 0.0 1.0"/>
+                <color rgba="1.0 0.65 0.0 1.0"/>
                 </material>
         </visual>
@@ -193,5 +193,5 @@
 <joint name="camera_joint" type="fixed">
         <preserveFixedJoint>true</preserveFixedJoint>
-        <origin rpy="0 0 0" xyz="0.0 0 0.2045" />
+        <origin rpy="0 0 0" xyz="0.1335 0 0.2045" />
         <parent link="robot_base_link" />
         <child link="camera_link" />
