Commit message: first version control diff_drive

File: src/mars_robot/urdf/mars_robot.urdf.xacro (robot description, xacro)
@@ -2,5 +2,52 @@
 <robot xmlns:xacro="http://www.ros.org/wiki/xacro" name="mars_robot">
 <xacro:include filename="mars_robot.gazebo" />
-<xacro:include filename="mars_robot.ros2_control.xacro" />
+<!-- <xacro:include filename="mars_robot.ros2_control.xacro" />  -->
+<ros2_control name="mars_robot_control" type="system">
+        <hardware>
+        <plugin>test_system</plugin>
+      <!--  <xacro:if value="${use_fake_hardware}">
+          <plugin>fake_components/GenericSystem</plugin>
+          <param name="fake_sensor_commands">${fake_sensor_commands}</param>
+          <param name="state_following_offset">0.0</param>
+        </xacro:if>
+        <xacro:unless value="${use_fake_hardware}">
+          <plugin>ros2_control_demo_hardware/DiffBotSystemHardware</plugin>
+          <param name="example_param_hw_start_duration_sec">2.0</param>
+          <param name="example_param_hw_stop_duration_sec">3.0</param>
+        </xacro:unless> -->
+        </hardware>
+        <joint name="front_left_wheel_joint">
+        <command_interface name="velocity">
+                <param name="min">-1</param>
+                <param name="max">1</param>
+        </command_interface>
+        <state_interface name="position"/>
+        <state_interface name="velocity"/>
+        </joint>
+        <joint name="front_right_wheel_joint">
+        <command_interface name="velocity">
+                <param name="min">-1</param>
+                <param name="max">1</param>
+        </command_interface>
+        <state_interface name="position"/>
+        <state_interface name="velocity"/>
+        </joint>
+        <joint name="rear_left_wheel_joint">
+        <command_interface name="velocity">
+                <param name="min">-1</param>
+                <param name="max">1</param>
+        </command_interface>
+        <state_interface name="position"/>
+        <state_interface name="velocity"/>
+        </joint>
+        <joint name="rear_right_wheel_joint">
+        <command_interface name="velocity">
+                <param name="min">-1</param>
+                <param name="max">1</param>
+        </command_interface>
+        <state_interface name="position"/>
+        <state_interface name="velocity"/>
+        </joint>
+</ros2_control>
 <!-- This first link, "world" is empty-->
 <link name="mars_robot_footprint"></link>

Commit message: Integrate robot_localization and orb_slam into mars_robot

File: src/mars_robot/urdf/mars_robot.urdf.xacro (robot description, xacro)
@@ -42,7 +42,7 @@
         </joint>
 </ros2_control>
-<!-- This first link, "world" is empty-->
-<link name="mars_robot_footprint"></link>
-<link name="robot_base_link">
+<!-- This first link, "base_footprint" is empty-->
+<!-- <link name="base_footprint"></link>         -->
+<link name="base_link">
         <visual>
                 <origin xyz="0 0 0.1115" rpy="0.0 0.0 0.0"/>
@@ -71,11 +71,10 @@
         </collision>
 </link>
-<!-- Fixed joint from "world" to "base"-->
-<joint name="base_joint" type="fixed">
-        <preserveFixedJoint>true</preserveFixedJoint>
-        <origin xyz="0.0 0 0.0615" rpy="0 0 0"/>
-        <parent link="mars_robot_footprint"/>
-        <child link="robot_base_link"/>
-</joint>
+<!-- Fixed joint from "base_footprint" to "base"-->
+<!-- <joint name="base_joint" type="fixed">
+        <origin xyz="0.0 0.0 0.0615" rpy="0 0 0"/>
+        <parent link="base_footprint"/>
+        <child link="base_link"/>
+</joint> -->
 <link name="front_left_wheel_link">
         <visual>
@@ -104,9 +103,8 @@
 </link>
 <joint name="front_left_wheel_joint" type="continuous">
-        <preserveFixedJoint>true</preserveFixedJoint>
-        <parent link="robot_base_link"/>
+        <parent link="base_link"/>
         <child link="front_left_wheel_link"/>
         <origin rpy="1.5708 0 0" xyz="0.0955 0.141 0"/>
-        <implicitSpringDamper>1</implicitSpringDamper>
+        <!-- <implicitSpringDamper>1</implicitSpringDamper> -->
 </joint>
 <link name="front_right_wheel_link">
@@ -136,6 +134,5 @@
 </link>
 <joint name="front_right_wheel_joint" type="continuous">
-        <preserveFixedJoint>true</preserveFixedJoint>
-        <parent link="robot_base_link"/>
+        <parent link="base_link"/>
         <child link="front_right_wheel_link"/>
         <origin rpy="1.5708 0 0" xyz="0.0955 -0.141 0"/>
@@ -168,6 +165,5 @@
 </link>
 <joint name="rear_left_wheel_joint" type="continuous">
-        <preserveFixedJoint>true</preserveFixedJoint>
-        <parent link="robot_base_link"/>
+        <parent link="base_link"/>
         <child link="rear_left_wheel_link"/>
         <origin rpy="1.5708 0 0" xyz="-0.0955 0.141 0"/>
@@ -200,6 +196,5 @@
 </link>
 <joint name="rear_right_wheel_joint" type="continuous">
-        <preserveFixedJoint>true</preserveFixedJoint>
-        <parent link="robot_base_link"/>
+        <parent link="base_link"/>
         <child link="rear_right_wheel_link"/>
         <origin rpy="1.5708 0 0" xyz="-0.0955 -0.141 0"/>
@@ -215,6 +210,5 @@
 </link>
 <joint name="imu_joint" type="fixed">
-        <preserveFixedJoint>true</preserveFixedJoint>
-        <parent link="robot_base_link" />
+        <parent link="base_link" />
         <child link="imu_link" />
         <origin rpy="0 0 0" xyz="0.0495 0.01 0.0665" />
@@ -232,7 +226,6 @@
 </link>
 <joint name="camera_joint" type="fixed">
-        <preserveFixedJoint>true</preserveFixedJoint>
         <origin rpy="0 0 0" xyz="0.1335 0 0.2045" />
-        <parent link="robot_base_link" />
+        <parent link="base_link" />
         <child link="camera_link" />
 </joint>
@@ -240,5 +233,4 @@
       so that ros and opencv can operate on the camera frame correctly -->
 <joint name="camera_optical_joint" type="fixed">
-        <preserveFixedJoint>true</preserveFixedJoint>
         <!-- these values have to be these values otherwise the gazebo camera image
         won't be aligned properly with the frame it is supposedly originating from -->

Commit message: Small changes Mars robot

File: src/mars_robot/urdf/mars_robot.urdf.xacro (robot description, xacro)
@@ -43,5 +43,5 @@
 </ros2_control>
 <!-- This first link, "base_footprint" is empty-->
-<!-- <link name="base_footprint"></link>         -->
+<link name="base_footprint"></link>
 <link name="base_link">
         <visual>
@@ -72,9 +72,9 @@
 </link>
 <!-- Fixed joint from "base_footprint" to "base"-->
-<!-- <joint name="base_joint" type="fixed">
+<joint name="base_joint" type="fixed">
         <origin xyz="0.0 0.0 0.0615" rpy="0 0 0"/>
         <parent link="base_footprint"/>
         <child link="base_link"/>
-</joint> -->
+</joint>
 <link name="front_left_wheel_link">
         <visual>
